Commit message: Add Lidar to URDF model

File: ros_ws/src/robot/description/robot_core.xacro (robot description, xacro)
@@ -13,4 +13,7 @@
     <material name="black">
         <color rgba="0 0 0 1"/>
+    </material>
+    <material name="grey" >
+        <color rgba="0.5725490196078431 0.5843137254901961 0.5686274509803921 1.0" />
     </material>
     <!-- BASE LINK -->
